Commit message: urdf model can now be loaded into rivz

File: src/simulation/urdf/simulation.urdf (robot description, URDF)
Before this commit: robot mycar, 1 links, 0 joints
Links:
- added link laser_link; visual cylinder length=0.02 radius=0.02
- link base_link: geometry visual cylinder length=0.12 radius=0.10
Joints:
- added joint laser_joint: type fixed, parent base_link, child laser_link, origin xyz=0 0 0.075
